File: STM32 Bluetooth Hardware Design.kicad_pcb (KiCad board)
At the start: 4 copper layers, 42 parts, among them J1 TC2030, J2 Conn_Coaxial, J3 USB_C_Receptacle_USB2.0_16P, J4 Conn_01x04_Pin, SW1 SW_Push, U1 STM32WB55CEUx, U2 USBLC6-2SC6, U3 MIC5365-3.3YD5, U4 USBLC6-2SC6, X1 32kHz, X2 32MHz

Commit message: added stuff
Parts:
- moved SW1 49.6 mm to (88.6, 104.8)
- moved J3 45.1 mm to (80.2, 96.8), turned to -90 degrees
- moved R4 39.6 mm to (87.0, 94.0), turned to 90 degrees
- moved U3 39.1 mm to (92.5, 93.5)
- moved R1 33.5 mm to (115.0, 104.5), turned to -90 degrees
- moved C8 31.4 mm to (121.5, 92.3), turned to 90 degrees
- moved C10 30.6 mm to (118.0, 95.0), turned to -90 degrees
- moved U2 28.5 mm to (92.0, 99.0), turned to 0 degrees
- moved R5 28.4 mm to (119.0, 101.6), turned to 90 degrees
- moved U4 28.2 mm to (128.6, 104.5)
- moved C12 27.8 mm to (111.5, 102.5)
- moved D1 25.9 mm to (119.0, 99.3), turned to 90 degrees
- moved C5 25.2 mm to (90.0, 88.4), turned to -90 degrees
- moved C13 24.8 mm to (109.0, 102.5), turned to 180 degrees
- moved C1 24.7 mm to (106.0, 88.5), turned to -90 degrees
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